File: LLv2_L/LLv2_L.kicad_pcb (KiCad board)
At the start: 2 copper layers, 128 x 107.4 mm, 10 parts, among them IC1 TEENSY_4.0, J1 AudioJack4

Commit message: Update Softwere
Parts:
- renumbered Home to Home1, Menu to Menu1, Start to Start1, ← to ←1, ↑ to ↑1, → to →1, ↓ to ↓1
Connections:
- net Net-(IC1-0) renamed RX
- net Net-(IC1-1) renamed TX
- net Net-(IC1-10) renamed 10pin
- net Net-(IC1-11) renamed 11pin
- net Net-(IC1-12) renamed 12pin
- net Net-(IC1-23) renamed 23pin
- net Net-(IC1-6) renamed 6pin
- net Net-(IC1-7) renamed 7pin
- net Net-(IC1-8) renamed 8pin
- net Net-(IC1-9) renamed 9pin
- net Net-(IC1-GND_1) renamed GND1
- net Net-(IC1-GND_2) renamed GND2
- net Net-(IC1-GND_3) renamed GND3
- net Net-(IC1-VIN_(3.6_TO_5.5_VOLTS)) renamed VIN
